File: PCB/PCB.kicad_pcb (KiCad board)
At the start: 2 copper layers, 88.2 x 105 mm, 32 parts, among them J1 Conn_01x10_Socket, J10 DMX-OUT, J2 Conn_01x06, J3 Screw_Terminal_01x02, J4 TEST_1P, J5 DMX-IN, J6 TEST_1P, Q1 BC847W, Q2 BC847W, Q3 BC847W, SW2 SW_Coded_SH-7010, U1 SP3485CN, U3 ESP32-WROOM

Commit message: add expansion port and level shifter in progress
Parts:
- removed J10: DMX-OUT, AC3MAH-AU-PRE:AC3MAH-AU-PRE
- removed SW2: SW_Coded_SH-7010, Button_Switch_THT:Nidec_SD-2011
- added C12: 10uF/100V, Capacitor_SMD:C_1210_3225Metric, F.Cu at (120.1, 66.1)
- added C13: 0.1uF, Capacitor_SMD:C_0603_1608Metric, F.Cu at (78.7, 60.7)
- added C14: 0.1uF, Capacitor_SMD:C_0603_1608Metric, F.Cu at (78.9, 54.1)
- added C15: 0.1uF, Capacitor_SMD:C_0603_1608Metric, F.Cu at (112.7, 72.2)
- added C16: 0.1uF, Capacitor_SMD:C_0603_1608Metric, F.Cu at (120.3, 72.2)
- added C6: 0.1uF, Capacitor_SMD:C_0603_1608Metric, F.Cu at (113.7, 100.9)
- added J7: Conn_01x08, Connector_PinHeader_2.54mm:PinHeader_1x08_P2.54mm_Horizontal, F.Cu at (128.4, 106.7)
- added J8: Conn_01x13, Connector_PinHeader_2.54mm:PinHeader_1x13_P2.54mm_Horizontal, F.Cu at (128.4, 62.3)
- added JP1: Jumper_3_Open, Connector_PinHeader_2.54mm:PinHeader_1x03_P2.54mm_Vertical, F.Cu at (73.1, 60.0)
- added JP2: Jumper_3_Open, Connector_PinHeader_2.54mm:PinHeader_1x03_P2.54mm_Vertical, F.Cu at (109.7, 87.2)
- added R2: 4.7k, Resistor_SMD:R_0603_1608Metric, F.Cu at (75.9, 126.5)
- added R7: 4.7k, Resistor_SMD:R_0603_1608Metric, F.Cu at (73.8, 126.4)
- added SW1: SW_DIP_x08, Button_Switch_THT:SW_DIP_SPSTx08_Piano_CTS_Series194-8MSTN_W7.62mm_P2.54mm, F.Cu at (47.2, 118.1)
- added U2: PCF8574, Package_SO:SSOP-20_4.4x6.5mm_P0.65mm, F.Cu at (66.2, 125.8)
- added U4: 74LVX3245TTR, Package_SO:TSSOP-24_4.4x7.8mm_P0.65mm, F.Cu at (85.5, 57.7)
- added U5: 74LVX3245TTR, Package_SO:TSSOP-24_4.4x7.8mm_P0.65mm, F.Cu at (116.5, 77.8)
- added U6: AMS1117-3.3, Package_TO_SOT_SMD:SOT-223-3_TabPin2, F.Cu at (118.4, 59.7)
- PS1: value TSR_0.6-4833WI -> TSR 0.6-4850WI
- moved C9 50.3 mm to (71.0, 124.5), turned to 90 degrees
- moved Q3 38.8 mm to (62.3, 60.9)
- moved R10 38.2 mm to (63.4, 66.2)
- moved R11 38.2 mm to (60.5, 66.2)
- moved C3 38.1 mm to (68.2, 110.9)
- moved U1 37.3 mm to (73.2, 107.2)
- moved C4 8.54 mm to (98.2, 77.3)
- moved C5 8.54 mm to (104.8, 77.3)
- moved PS1 8.07 mm to (99.5, 67.3)
- moved C1 6.49 mm to (74.5, 54.0)
- moved R5 6.49 mm to (70.7, 54.0)
- moved J5 2.18 mm to (44.1, 104.5)
- moved C2 1.33 mm to (74.5, 55.7)
- moved R6 1.33 mm to (70.7, 55.7)
Connections:
- net /HOME_POT renamed /START_POT
- net /LIMIT_POT renamed /END_POT
- net /XLR_DMX_2 renamed /DMX/XLR_DMX_2
- net /XLR_DMX_3 renamed /DMX/XLR_DMX_3
- C1 pad 1: /LIMIT_SWITCH -> /END_SWITCH
- C2 pad 1: /HOME_SWITCH -> /START_SWITCH
- C5 pad 1: +3V3 -> +5V
- J1 pad 10: /LIMIT_SWITCH -> /START_SWITCH
- J1 pad 2: /EA+ -> /EB+
- J1 pad 3: /EB+ -> /EA+
- J1 pad 4: /ENA- -> /Shifter level stepper/B4
- J1 pad 5: +3V3 -> /Shifter level stepper/B3
- J1 pad 6: /DIR+ -> /Shifter level stepper/B2
- J1 pad 7: /PUL+ -> /Shifter level stepper/B1
- J1 pad 9: /HOME_SWITCH -> /END_SWITCH
- PS1 pad 3: +3V3 -> +5V
- R5 pad 1: /LIMIT_SWITCH -> /END_SWITCH
- R6 pad 1: /HOME_SWITCH -> /START_SWITCH
- U3 pad 13: unconnected-(U3-IO14-Pad13) -> /IO14
- U3 pad 14: unconnected-(U3-IO12-Pad14) -> /IO12
- U3 pad 16: unconnected-(U3-IO13-Pad16) -> /IO13
- U3 pad 17: unconnected-(U3-SD2/IO9-Pad17) -> /SD2
- U3 pad 18: unconnected-(U3-SD3/IO10-Pad18) -> /SD3
- U3 pad 19: unconnected-(U3-CMD/IO11-Pad19) -> /CMD
- U3 pad 20: unconnected-(U3-CLK/IO6-Pad20) -> /CLK
- U3 pad 21: unconnected-(U3-SD0/IO7-Pad21) -> /SD0
- U3 pad 22: unconnected-(U3-SD1/IO8-Pad22) -> /SD1
- U3 pad 23: unconnected-(U3-IO15-Pad23) -> /IO15
- U3 pad 24: unconnected-(U3-IO2-Pad24) -> /IO_2
- U3 pad 29: /ADR8 -> /EA+
- U3 pad 30: /ADR4 -> /EB+
- U3 pad 31: /ADR2 -> /IO19
- U3 pad 33: /ADR1 -> /SDA
- U3 pad 36: /EA+ -> /SCL
- U3 pad 37: /EB+ -> /IO23
- U3 pad 6: /LIMIT_SWITCH -> /START_SWITCH
- U3 pad 7: /HOME_SWITCH -> /END_SWITCH
- U3 pad 8: unconnected-(U3-IO32-Pad8) -> /IO32_One-wire
- U3 pad 9: unconnected-(U3-IO33-Pad9) -> /IO33
Routing:
- net /SDA: track 0.00 -> 161.1 mm, vias 0 -> 1
- net /SCL: track 0.00 -> 139.8 mm
- net +5V: track 0.00 -> 138.1 mm
- net +3V3: track 293.5 -> 381.5 mm, vias 2 -> 0
- net /START_SWITCH: track 0.00 -> 87.6 mm, vias 0 -> 1
- net /LIMIT_SWITCH: track 85.5 -> 0.00 mm
- net /HOME_SWITCH: track 83.8 -> 0.00 mm
- net /END_SWITCH: track 0.00 -> 78.5 mm, vias 0 -> 1
- net /IO23: track 0.00 -> 75.3 mm
- net /ADR1: track 74.9 -> 0.00 mm
- net /ADR4: track 65.6 -> 0.00 mm
- net /ESP32_BOOT: track 28.7 -> 93.7 mm
- net /ADR8: track 63.5 -> 0.00 mm
- net /ADR2: track 61.4 -> 0.00 mm, vias 1 -> 0
- net /IO15: track 0.00 -> 54.2 mm, vias 0 -> 2
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Other:
- board text added: "+3V3 IO_33 IO_32 IO_23 IO_19 IO_15 IO_14 IO_13 IO_12 IO_02 SCL SDA GND"
- board text added: "+3V3 SD2 SD3 CMD CLK SD0 SD1 GND"
- board text added: "DMX / OSC ESP Stepper controler Clément SAILLANT 09/2023 c.saillant@gmail.com"
- board text added: "Expansion port"
- board text added: "Internal Flash connection"
- board text added: "Isaac is the best"
- board text added: "lisael was awesome"
- board text added: "v0.05"
- board text removed: "Orphéo V0.5a 09/2023"
